Commit message: "commit"

File: trixy.xacro (robot description, xacro)
@@ -41,10 +41,9 @@
     <axis xyz="0 1 0"/>
   </joint>
-  <joint name="GPS_joint" type="fixed">
-    <origin xyz="0 0 0.005" rpy="0 0 0" />
-    <parent link="chassis"/>
-    <child link="gps_link" />
-    <axis xyz="0 1 0"/>
-  </joint>
+  <joint name="gps_joint" type="fixed">
+            <parent link="chassis"/>
+            <origin xyz="-0.06 0 0.115" rpy="0 0 0"/>
+            <child link="gps_link"/>
+        </joint>
   <joint name="left_camera_frame" type="fixed">
     <origin xyz="0 0.10 0.13" rpy="0 0 0" />
@@ -54,5 +53,5 @@
   </joint>
   <joint name="hokuyo_joint" type="fixed">
-    <origin xyz="0.2 0.1 0.1" rpy="0 0 0" />
+    <origin xyz="0.2 0.2 0.1" rpy="0 0 0" />
     <parent link="chassis"/>
     <child link="hokuyo" />
@@ -184,25 +183,25 @@
   </link>
   <link name="gps_link">
-    <collision>
-      <origin xyz="0 0 0.1" rpy="0 0 0"/>
-      <geometry>
-        <box size="0.1 0.1 0.1"/>
-      </geometry>
-    </collision>
-    <visual>
-      <origin xyz="0 0 0.1" rpy="0 0 0"/>
-      <geometry>
-        <cylinder radius="0.05" length="0.05"/>
-      </geometry>
-    </visual>
-    <inertial>
-      <origin xyz="0 0 0.1" rpy="0 0 0"/>
-      <mass value="1"/>
-      <inertia
-        ixx="1.0" ixy="0.0" ixz="0.0"
-        iyy="1.0" iyz="0.0"
-        izz="1.0"/>
-    </inertial>
-  </link>
+        <collision>
+        <origin xyz="0 0 0" rpy="0 0 0"/>
+        <geometry>
+            <box size="0.025 0.025 0.025"/>
+        </geometry>
+        </collision>
+        <visual>
+        <origin xyz="0 0 0" rpy="0 0 0"/>
+        <geometry>
+            <box size="0.025 0.025 0.025"/>
+        </geometry>
+        </visual>
+        <inertial>
+        <origin xyz="0 0 1" rpy="0 0 0"/>
+        <mass value="1"/>
+        <inertia
+            ixx="1.0" ixy="0.0" ixz="0.0"
+            iyy="1.0" iyz="0.0"
+            izz="1.0"/>
+        </inertial>
+    </link>
   <link name="left_wheel_2">
     <inertial>

Commit message: Add files via upload

File: trixy.xacro (robot description, xacro)
@@ -59,10 +59,10 @@
   </joint>
   <joint type="continuous" name="left_wheel_hinge">
-    <origin xyz="-0.1 0.30 0" rpy="0 0 0" />
+    <origin xyz="-0.12 0.30 0" rpy="0 0 0" />
     <parent link="chassis"/>
     <child link="left_wheel" />
     <axis xyz="0 1 0" rpy="0 0 0" />
     <limit effort="10000" velocity="1000" />
-    <dynamics damping="1.0" friction="1.0" />
+    <dynamics damping="1.0" friction="1.0000" />
   </joint>
   <joint type="continuous" name="right_wheel_hinge">
@@ -72,13 +72,13 @@
     <axis xyz="0 1 0" rpy="0 0 0" />
     <limit effort="10000" velocity="1000" />
-    <dynamics damping="1.0" friction="1.0" />
+    <dynamics damping="1.0" friction="1.0000" />
   </joint>
   <joint type="continuous" name="right_wheel_hinge_2">
-  <origin xyz="-0.1 -0.30 0" rpy="0 0 0" />
+  <origin xyz="-0.12 -0.30 0" rpy="0 0 0" />
   <parent link="chassis"/>
   <child link="right_wheel_2" />
   <axis xyz="0 1 0" rpy="0 0 0" />
   <limit effort="10000" velocity="1000" />
-  <dynamics damping="1.0" friction="1.0" />
+  <dynamics damping="1.0" friction="1.0000" />
 </joint>
 <joint type="continuous" name="left_wheel_hinge_2">
@@ -88,5 +88,5 @@
   <axis xyz="0 1 0" rpy="0 0 0" />
   <limit effort="10000" velocity="1000" />
-  <dynamics damping="1.0" friction="1.0" />
+  <dynamics damping="1.0" friction="1.00000" />
 </joint>
 <link name="camera">
@@ -205,4 +205,8 @@
     </link>
   <link name="left_wheel_2">
+  <mu1>0.5</mu1>
+    <mu2>0.5</mu2>
+    <kp>1000.0</kp>
+    <kd>1.0</kd>
     <inertial>
       <mass value="10"/>
@@ -228,4 +232,8 @@
   </link>
   <link name="left_wheel">
+    <mu1>0.5</mu1>
+    <mu2>0.5</mu2>
+    <kp>1000.0</kp>
+    <kd>1.0</kd>
     <inertial>
       <mass value="10"/>
@@ -251,4 +259,8 @@
   </link>
   <link name="right_wheel">
+  <mu1>0.5</mu1>
+    <mu2>0.5</mu2>
+    <kp>1000.0</kp>
+    <kd>1.0</kd>
     <inertial>
       <mass value="10"/>
@@ -274,4 +286,8 @@
   </link>
   <link name="right_wheel_2">
+  <mu1>0.5</mu1>
+    <mu2>0.5</mu2>
+    <kp>1000.0</kp>
+    <kd>1.0</kd>
   <inertial>
     <mass value="10"/>
